File: main.kicad_sch (KiCad schematic)
At the start: 60 parts, among them J13 Conn_01x03_Socket, J14 Conn_01x01_Female

Commit message: Added serial number field
Other:
- note added: "TODO: - Test hot into short"
- note removed: "TODO: - Add serial number - Test hot into short"
Changed lines of the file:
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@@
     (effects (font (size 1.27 1.27)) (justify left bottom))
   )
-  (text "TODO:\n- Add serial number\n- Test hot into short" (at 109.22 57.15 0)
+  (text "TODO:\n- Test hot into short" (at 109.22 57.15 0)
     (effects (font (size 1.27 1.27)) (justify left bottom))
   )
