File: main.kicad_sch (KiCad schematic)
At the start: 60 parts, among them J13 Conn_01x03_Socket, J14 Conn_01x01_Female

Commit message: Updated libs
Parts:
- LOGO2: symbol Custom_logos:Logo_RoHS -> Custom_logos:SYM_RoHS
Changed lines of the file:
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@@
     )
   )
-  (symbol (lib_id "Custom_logos:Logo_APQ") (at 242.57 171.45 0) (unit 1)
+  (symbol (lib_id "Custom_logos:Logo_APQ") (at 255.27 171.45 0) (unit 1)
     (in_bom no) (on_board yes) (dnp no)
-    (property "Reference" "LOGO1" (at 248.92 164.465 0)
-      (effects (font (size 1.27 1.27)) hide)
-    )
-    (property "Value" "Logo_APQ" (at 248.92 177.8 0)
-      (effects (font (size 1.27 1.27)) hide)
-    )
-    (property "Footprint" "Custom_footprints_project:APQ-Logo_small" (at 250.19 171.45 0)
-      (effects (font (size 1.27 1.27)) hide)
-    )
-    (property "Datasheet" "~" (at 250.19 171.45 0)
-      (effects (font (size 1.27 1.27)) hide)
-    )
-    (property "MFN" "" (at 242.57 171.45 0)
-      (effects (font (size 1.27 1.27)) hide)
-    )
-    (property "PN" "" (at 242.57 171.45 0)
-      (effects (font (size 1.27 1.27)) hide)
-    )
-    (property "RoHS" "" (at 242.57 171.45 0)
-      (effects (font (size 1.27 1.27)) hide)
-    )
-    (property "Sim.Enable" "0" (at 242.57 171.45 0)
+    (property "Reference" "LOGO1" (at 261.62 164.465 0)
+      (effects (font (size 1.27 1.27)) hide)
+    )
+    (property "Value" "Logo_APQ" (at 261.62 177.8 0)
+      (effects (font (size 1.27 1.27)) hide)
+    )
+    (property "Footprint" "Custom_footprints_project:APQ-Logo_small" (at 262.89 171.45 0)
+      (effects (font (size 1.27 1.27)) hide)
+    )
+    (property "Datasheet" "~" (at 262.89 171.45 0)
+      (effects (font (size 1.27 1.27)) hide)
+    )
+    (property "MFN" "" (at 255.27 171.45 0)
+      (effects (font (size 1.27 1.27)) hide)
+    )
+    (property "PN" "" (at 255.27 171.45 0)
+      (effects (font (size 1.27 1.27)) hide)
+    )
+    (property "RoHS" "" (at 255.27 171.45 0)
+      (effects (font (size 1.27 1.27)) hide)
+    )
+    (property "Sim.Enable" "0" (at 255.27 171.45 0)
       (effects (font (size 1.27 1.27)) hide)
     )
@@
     )
   )
-  (symbol (lib_id "Custom_logos:Logo_RoHS") (at 209.55 170.18 0) (unit 1)
-    (in_bom no) (on_board yes) (dnp no) (fields_autoplaced)
-    (property "Reference" "LOGO2" (at 215.9 163.195 0)
-      (effects (font (size 1.27 1.27)) hide)
-    )
-    (property "Value" "Logo_RoHS" (at 215.9 176.53 0)
-      (effects (font (size 1.27 1.27)) hide)
-    )
-    (property "Footprint" "Symbol:RoHS-Logo_6mm_SilkScreen" (at 217.17 170.18 0)
-      (effects (font (size 1.27 1.27)) hide)
-    )
-    (property "Datasheet" "~" (at 217.17 170.18 0)
-      (effects (font (size 1.27 1.27)) hide)
-    )
-    (property "MFN" "" (at 209.55 170.18 0)
-      (effects (font (size 1.27 1.27)) hide)
-    )
-    (property "PN" "" (at 209.55 170.18 0)
-      (effects (font (size 1.27 1.27)) hide)
-    )
-    (property "Sim.Enable" "0" (at 209.55 170.18 0)
-      (effects (font (size 1.27 1.27)) hide)
-    )
-    (property "RoHS" "" (at 209.55 170.18 0)
-      (effects (font (size 1.27 1.27)) hide)
-    )
+  (symbol (lib_id "Custom_logos:SYM_RoHS") (at 223.52 170.18 0) (unit 1)
+    (in_bom no) (on_board no) (dnp no) (fields_autoplaced)
+    (property "Reference" "LOGO2" (at 229.87 163.195 0)
+      (effects (font (size 1.27 1.27)) hide)
+    )
+    (property "Value" "Logo_RoHS" (at 229.87 176.53 0)
+      (effects (font (size 1.27 1.27)) hide)
+    )
+    (property "Footprint" "Symbol:RoHS-Logo_6mm_SilkScreen" (at 231.14 170.18 0)
+      (effects (font (size 1.27 1.27)) hide)
+    )
+    (property "Datasheet" "~" (at 223.52 170.18 0)
+      (effects (font (size 1.27 1.27)) hide)
+    )
+    (property "MFN" "" (at 223.52 170.18 0)
+      (effects (font (size 1.27 1.27)) hide)
+    )
+    (property "PN" "" (at 223.52 170.18 0)
+      (effects (font (size 1.27 1.27)) hide)
+    )
+    (property "Sim.Enable" "0" (at 223.52 170.18 0)
+      (effects (font (size 1.27 1.27)) hide)
+    )
+    (property "RoHS" "" (at 223.52 170.18 0)
+      (effects (font (size 1.27 1.27)) hide)
+    )
